File: SIMM/Hardware/Tarjeta hija/Esquematicos/SIMM.sch (KiCad schematic (older format))
At the start: 38 parts, among them J1 JACK_3P, J2 USB_2, J3 USB-MINI, K1 CONN_3, P1 CONN_12X2, P2 CONN_12X2, P3 CONN_20X2, P4 CONN_12X2, P5 GPS SKYLAB, P6 CONN_2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

Commit message: mar 27 /13
Parts:
- removed K1: CONN_3, symbol CONN_3
- added P9: Bluetooth, symbol CONN_4
Connections:
- wire segments 216 -> 218
Changed lines of the file:
@@
 LIBS:logo1
 LIBS:SIMM-cache
-EELAYER 27 0
+EELAYER 24 0
 EELAYER END
 $Descr A3 16535 11693
@@
 	4850 1500 3850 1500
 Wire Wire Line
-	14450 3250 14050 3250
-Wire Wire Line
-	14350 3550 14350 3350
-Wire Wire Line
-	14350 3350 14450 3350
+	14000 3550 13600 3550
+Wire Wire Line
+	13300 3550 13300 3350
+Wire Wire Line
+	13300 3350 14000 3350
 Wire Wire Line
 	2550 3100 3350 3100
@@
 	2550 3200 3350 3200
 Wire Wire Line
-	14450 3150 14050 3150
+	14000 3450 13600 3450
 Wire Wire Line
 	3850 1200 4850 1200
@@
 VDAC1
 $Comp
-L GND #PWR01
+L GND #PWR15
 U 1 1 51E80379
 P 7500 7500
-F 0 "#PWR01" H 7500 7500 30  0001 C CNN
+F 0 "#PWR15" H 7500 7500 30  0001 C CNN
 F 1 "GND" H 7500 7430 30  0001 C CNN
 F 2 "" H 7500 7500 60  0001 C CNN
@@
 	1    0    0    -1
 $EndComp
-Text Label 14050 3250 0    60   ~ 0
+Text Label 13600 3550 0    60   ~ 0
 TX
-Text Label 14050 3150 0    60   ~ 0
+Text Label 13600 3450 0    60   ~ 0
 RX
 $Comp
-L GND #PWR02
+L GND #PWR25
 U 1 1 51E7F8AF
-P 14350 3550
-F 0 "#PWR02" H 14350 3550 30  0001 C CNN
-F 1 "GND" H 14350 3480 30  0001 C CNN
-F 2 "" H 14350 3550 60  0001 C CNN
-F 3 "" H 14350 3550 60  0001 C CNN
-	1    14350 3550
-	1    0    0    -1
-$EndComp
-$Comp
-L CONN_3 K1
-U 1 1 51E7F89B
-P 14800 3250
-F 0 "K1" V 14750 3250 50  0000 C CNN
-F 1 "CONN_3" V 14850 3250 40  0000 C CNN
-F 2 "" H 14800 3250 60  0001 C CNN
-F 3 "" H 14800 3250 60  0001 C CNN
-	1    14800 3250
+P 13300 3550
+F 0 "#PWR25" H 13300 3550 30  0001 C CNN
+F 1 "GND" H 13300 3480 30  0001 C CNN
+F 2 "" H 13300 3550 60  0001 C CNN
+F 3 "" H 13300 3550 60  0001 C CNN
+	1    13300 3550
 	1    0    0    -1
 $EndComp
@@
 $EndComp
 $Comp
-L GND #PWR03
+L GND #PWR30
 U 1 1 51E6DF73
 P 14750 5350
-F 0 "#PWR03" H 14750 5350 30  0001 C CNN
+F 0 "#PWR30" H 14750 5350 30  0001 C CNN
 F 1 "GND" H 14750 5280 30  0001 C CNN
 F 2 "" H 14750 5350 60  0001 C CNN
@@
 $EndComp
 $Comp
-L GND #PWR04
+L GND #PWR24
 U 1 1 51E6DE1D
 P 12600 5350
-F 0 "#PWR04" H 12600 5350 30  0001 C CNN
+F 0 "#PWR24" H 12600 5350 30  0001 C CNN
 F 1 "GND" H 12600 5280 30  0001 C CNN
 F 2 "" H 12600 5350 60  0001 C CNN
@@
 $EndComp
 $Comp
-L +5V #PWR05
+L +5V #PWR28
 U 1 1 51E6DE08
 P 14300 4400
-F 0 "#PWR05" H 14300 4490 20  0001 C CNN
+F 0 "#PWR28" H 14300 4490 20  0001 C CNN
 F 1 "+5V" H 14300 4490 30  0000 C CNN
 F 2 "" H 14300 4400 60  0001 C CNN
@@
 $EndComp
 $Comp
-L AGND #PWR06
+L AGND #PWR23
 U 1 1 51E6DDE7
 P 12050 5250
-F 0 "#PWR06" H 12050 5250 40  0001 C CNN
+F 0 "#PWR23" H 12050 5250 40  0001 C CNN
 F 1 "AGND" H 12050 5180 50  0000 C CNN
 F 2 "" H 12050 5250 60  0001 C CNN
@@
 $EndComp
 $Comp
-L GND #PWR07
+L GND #PWR29
 U 1 1 51E6DD9E
 P 14300 5350
-F 0 "#PWR07" H 14300 5350 30  0001 C CNN
+F 0 "#PWR29" H 14300 5350 30  0001 C CNN
 F 1 "GND" H 14300 5280 30  0001 C CNN
 F 2 "" H 14300 5350 60  0001 C CNN
@@
 $EndComp
 $Comp
-L GND #PWR08
+L GND #PWR26
 U 1 1 51E6DD9B
 P 13450 5350
-F 0 "#PWR08" H 13450 5350 30  0001 C CNN
+F 0 "#PWR26" H 13450 5350 30  0001 C CNN
 F 1 "GND" H 13450 5280 30  0001 C CNN
 F 2 "" H 13450 5350 60  0001 C CNN
@@
 $EndComp
 $Comp
-L 3V3 #PWR09
+L 3V3 #PWR12
 U 1 1 51E6DD06
 P 6700 900
-F 0 "#PWR09" H 6700 1000 40  0001 C CNN
+F 0 "#PWR12" H 6700 1000 40  0001 C CNN
 F 1 "3V3" H 6700 1025 40  0000 C CNN
 F 2 "" H 6700 900 60  0001 C CNN
@@
 $EndComp
 $Comp
-L 3V3 #PWR010
+L 3V3 #PWR7
 U 1 1 51E6CD87
 P 3900 5350
-F 0 "#PWR010" H 3900 5450 40  0001 C CNN
+F 0 "#PWR7" H 3900 5450 40  0001 C CNN
 F 1 "3V3" H 3900 5475 40  0000 C CNN
 F 2 "" H 3900 5350 60  0001 C CNN
@@
 NoConn ~ 2300 5850
 $Comp
-L GND #PWR011
+L GND #PWR4
 U 1 1 51E6CC05
 P 3350 5850
-F 0 "#PWR011" H 3350 5850 30  0001 C CNN
+F 0 "#PWR4" H 3350 5850 30  0001 C CNN
 F 1 "GND" H 3350 5780 30  0001 C CNN
 F 2 "" H 3350 5850 60  0001 C CNN
@@
 $EndComp
 $Comp
-L 3V3 #PWR012
+L 3V3 #PWR3
 U 1 1 51E6CBE5
 P 2500 5050
-F 0 "#PWR012" H 2500 5150 40  0001 C CNN
+F 0 "#PWR3" H 2500 5150 40  0001 C CNN
 F 1 "3V3" H 2500 5175 40  0000 C CNN
 F 2 "" H 2500 5050 60  0001 C CNN
@@
 LCD_D0
 $Comp
-L GND #PWR013
+L GND #PWR2
 U 1 1 51E6ABD9
 P 1800 1150
-F 0 "#PWR013" H 1800 1150 30  0001 C CNN
+F 0 "#PWR2" H 1800 1150 30  0001 C CNN
 F 1 "GND" H 1800 1080 30  0001 C CNN
 F 2 "" H 1800 1150 60  0001 C CNN
@@
 $EndComp
 $Comp
-L 3V3 #PWR014
+L 3V3 #PWR1
 U 1 1 51E6ABAB
 P 1150 1200
-F 0 "#PWR014" H 1150 1300 40  0001 C CNN
+F 0 "#PWR1" H 1150 1300 40  0001 C CNN
 F 1 "3V3" H 1150 1325 40  0000 C CNN
 F 2 "" H 1150 1200 60  0001 C CNN
@@
 PA17
 $Comp
-L 3V3 #PWR015
+L 3V3 #PWR5
 U 1 1 51E5BC39
 P 3350 7500
-F 0 "#PWR015" H 3350 7600 40  0001 C CNN
+F 0 "#PWR5" H 3350 7600 40  0001 C CNN
 F 1 "3V3" H 3350 7625 40  0000 C CNN
 F 2 "" H 3350 7500 60  0001 C CNN
@@
 $EndComp
 $Comp
-L GND #PWR016
+L GND #PWR6
 U 1 1 51E5BC2E
 P 3500 10050
-F 0 "#PWR016" H 3500 10050 30  0001 C CNN
+F 0 "#PWR6" H 3500 10050 30  0001 C CNN
 F 1 "GND" H 3500 9980 30  0001 C CNN
 F 2 "" H 3500 10050 60  0001 C CNN
@@
 $EndComp
 $Comp
-L 3V3 #PWR017
+L 3V3 #PWR11
 U 1 1 51E57824
 P 6400 4600
-F 0 "#PWR017" H 6400 4700 40  0001 C CNN
+F 0 "#PWR11" H 6400 4700 40  0001 C CNN
 F 1 "3V3" H 6400 4725 40  0000 C CNN
 F 2 "" H 6400 4600 60  0001 C CNN
@@
 $EndComp
 $Comp
-L 3V3 #PWR018
+L 3V3 #PWR13
 U 1 1 51E5781F
 P 7100 4600
-F 0 "#PWR018" H 7100 4700 40  0001 C CNN
+F 0 "#PWR13" H 7100 4700 40  0001 C CNN
 F 1 "3V3" H 7100 4725 40  0000 C CNN
 F 2 "" H 7100 4600 60  0001 C CNN
@@
 $EndComp
 $Comp
-L 3V3 #PWR019
+L 3V3 #PWR17
 U 1 1 51E57812
 P 8200 4600
-F 0 "#PWR019" H 8200 4700 40  0001 C CNN
+F 0 "#PWR17" H 8200 4700 40  0001 C CNN
 F 1 "3V3" H 8200 4725 40  0000 C CNN
 F 2 "" H 8200 4600 60  0001 C CNN
@@
 $EndComp
 $Comp
-L 3V3 #PWR020
+L 3V3 #PWR18
 U 1 1 51E573BB
 P 9000 4600
-F 0 "#PWR020" H 9000 4700 40  0001 C CNN
+F 0 "#PWR18" H 9000 4700 40  0001 C CNN
 F 1 "3V3" H 9000 4725 40  0000 C CNN
 F 2 "" H 9000 4600 60  0001 C CNN
@@
 USB_5V
 $Comp
-L +5V #PWR021
+L +5V #PWR22
 U 1 1 51E56FAA
 P 10950 6800
-F 0 "#PWR021" H 10950 6890 20  0001 C CNN
+F 0 "#PWR22" H 10950 6890 20  0001 C CNN
 F 1 "+5V" H 10950 6890 30  0000 C CNN
 F 2 "" H 10950 6800 60  0001 C CNN
@@
 USB_DM
 $Comp
-L GND #PWR022
+L GND #PWR20
 U 1 1 51E2C141
 P 10500 9900
-F 0 "#PWR022" H 10500 9900 30  0001 C CNN
+F 0 "#PWR20" H 10500 9900 30  0001 C CNN
 F 1 "GND" H 10500 9830 30  0001 C CNN
 F 2 "" H 10500 9900 60  0001 C CNN
@@
 $EndComp
 $Comp
-L GND #PWR023
+L GND #PWR31
 U 1 1 51E2C13C
 P 14850 9350
-F 0 "#PWR023" H 14850 9350 30  0001 C CNN
+F 0 "#PWR31" H 14850 9350 30  0001 C CNN
 F 1 "GND" H 14850 9280 30  0001 C CNN
 F 2 "" H 14850 9350 60  0001 C CNN
@@
 $EndComp
 $Comp
-L GND #PWR024
+L GND #PWR21
 U 1 1 51E2C109
 P 10600 3500
-F 0 "#PWR024" H 10600 3500 30  0001 C CNN
+F 0 "#PWR21" H 10600 3500 30  0001 C CNN
 F 1 "GND" H 10600 3430 30  0001 C CNN
 F 2 "" H 10600 3500 60  0001 C CNN
@@
 $EndComp
 $Comp
-L GND #PWR025
+L GND #PWR14
 U 1 1 51E2C108
 P 7150 3450
-F 0 "#PWR025" H 7150 3450 30  0001 C CNN
+F 0 "#PWR14" H 7150 3450 30  0001 C CNN
 F 1 "GND" H 7150 3380 30  0001 C CNN
 F 2 "" H 7150 3450 60  0001 C CNN
@@
 $EndComp
 $Comp
-L 3V3 #PWR026
+L 3V3 #PWR19
 U 1 1 51E2C107
 P 9750 1950
-F 0 "#PWR026" H 9750 2050 40  0001 C CNN
+F 0 "#PWR19" H 9750 2050 40  0001 C CNN
 F 1 "3V3" H 9750 2075 40  0000 C CNN
 F 2 "" H 9750 1950 60  0001 C CNN
@@
 $EndComp
 $Comp
-L 3V3 #PWR027
+L 3V3 #PWR16
 U 1 1 51E2C106
 P 8050 1950
-F 0 "#PWR027" H 8050 2050 40  0001 C CNN
+F 0 "#PWR16" H 8050 2050 40  0001 C CNN
 F 1 "3V3" H 8050 2075 40  0000 C CNN
 F 2 "" H 8050 1950 60  0001 C CNN
@@
 $EndComp
 $Comp
-L +5V #PWR028
+L +5V #PWR8
 U 1 1 51E2C105
 P 4700 2750
-F 0 "#PWR028" H 4700 2840 20  0001 C CNN
+F 0 "#PWR8" H 4700 2840 20  0001 C CNN
 F 1 "+5V" H 4700 2840 30  0000 C CNN
 F 2 "" H 4700 2750 60  0001 C CNN
@@
 $EndComp
 $Comp
-L GND #PWR029
+L GND #PWR10
 U 1 1 51E2C104
 P 6100 900
-F 0 "#PWR029" H 6100 900 30  0001 C CNN
+F 0 "#PWR10" H 6100 900 30  0001 C CNN
 F 1 "GND" H 6100 830 30  0001 C CNN
 F 2 "" H 6100 900 60  0001 C CNN
@@
 $EndComp
 $Comp
-L +5V #PWR030
+L +5V #PWR9
 U 1 1 51E2C103
 P 4750 950
-F 0 "#PWR030" H 4750 1040 20  0001 C CNN
+F 0 "#PWR9" H 4750 1040 20  0001 C CNN
 F 1 "+5V" H 4750 1040 30  0000 C CNN
 F 2 "" H 4750 950 60  0001 C CNN
@@
 Connection ~ 14850 9150
 $Comp
-L GND #PWR031
+L GND #PWR32
 U 1 1 520FBF5E
 P 15050 7850
-F 0 "#PWR031" H 15050 7850 30  0001 C CNN
+F 0 "#PWR32" H 15050 7850 30  0001 C CNN
 F 1 "GND" H 15050 7780 30  0001 C CNN
 F 2 "" H 15050 7850 60  0000 C CNN
@@
 Connection ~ 14850 7500
 $Comp
-L LOGO #G?
+L LOGO #G1
 U 1 1 5212C235
 P 11200 10700
-F 0 "#G?" H 11200 10420 60  0001 C CNN
+F 0 "#G1" H 11200 10420 60  0001 C CNN
 F 1 "LOGO" H 11200 10980 60  0001 C CNN
 F 2 "" H 11200 10700 60  0000 C CNN
@@
 	1    0    0    -1
 $EndComp
+$Comp
+L CONN_4 P9
+U 1 1 5243EE4D
+P 14350 3400
+F 0 "P9" V 14300 3400 50  0000 C CNN
+F 1 "Bluetooth" V 14400 3400 50  0000 C CNN
+F 2 "" H 14350 3400 60  0000 C CNN
+F 3 "" H 14350 3400 60  0000 C CNN
+	1    14350 3400
+	1    0    0    -1
+$EndComp
+$Comp
+L 3V3 #PWR27
+U 1 1 5243F174
+P 13800 3150
+F 0 "#PWR27" H 13800 3250 40  0001 C CNN
+F 1 "3V3" H 13800 3275 40  0000 C CNN
+F 2 "" H 13800 3150 60  0000 C CNN
+F 3 "" H 13800 3150 60  0000 C CNN
+	1    13800 3150
+	1    0    0    -1
+$EndComp
+Wire Wire Line
+	14000 3250 13800 3250
+Wire Wire Line
+	13800 3250 13800 3150
 $EndSCHEMATC
